Commit message: Fix TF tree gap between FAST-LIO and vehicle; successfully tested flight

File: config/iris_vlp16.urdf (robot description, URDF)
Before this commit: robot iris_vlp16, 2 links, 1 joints
Links:
- added link body
Joints:
- added joint body_to_base_link_joint: type fixed, parent body, child base_link, origin xyz=0 0 0 rpy=0 0 0

Commit message: fix: De-duplicate EKF2 vision sources, fix ROS TF tree topology, align LiDAR extrinsics to 0.12m, and correct MAVROS ENU frame mapping in Flight Envelope Guard

File: config/iris_vlp16.urdf (robot description, URDF)
Before this commit: robot iris_vlp16, 3 links, 2 joints
Joints:
- joint velodyne_joint: origin xyz=0 0 0.08 rpy=0 0 0 -> xyz=0 0 0.12 rpy=0 0 0
